File: First/Work/project/Module_4/Module_4.kicad_pcb (KiCad board)
At the start: 2 copper layers, 76.2 x 113.3 mm, 12 parts

Commit message: Поправлена шелкография проекта
Parts:
- removed the REF** at (102.9, 101.6)
- added J3: Conn_01x10_Female, module_4:plc_x10, F.Cu at (102.9, 101.6)
- added SW1: SW_Push, module_4:button, F.Cu at (91.4, 26.0)
- A2: renamed from REF**; value Arduino_Nano -> Arduino_Nano_v3.x
- A3: renamed from REF**; value ZS-042 -> ZS-042_RTC1; footprint module_4:ZS-042 -> module_4:ZS-042_1
- J1: renamed from REF**; value klemmnik_x20 -> Conn_01x20
- J2, J5: renamed from REF**; value plc_x8 -> Conn_01x08_Female
- J4: renamed from REF**; value plc_x6 -> Conn_01x06_Female
- renumbered REF** to A1
Connections:
- A1 pad 1: (no net) -> /In+
- A1 pad 2: (no net) -> /In-
- A1 pad 3: (no net) -> /vin
- A1 pad 4: (no net) -> /gnd
- A2 pad 1: (no net) -> Net-(A2-Pad1)
- A2 pad 10: (no net) -> /d7
- A2 pad 11: (no net) -> /d8
- A2 pad 12: (no net) -> /d9
- A2 pad 13: (no net) -> /d10
- A2 pad 14: (no net) -> Net-(A2-Pad14)
- A2 pad 15: (no net) -> Net-(A2-Pad15)
- A2 pad 16: (no net) -> Net-(A2-Pad16)
- A2 pad 17: (no net) -> Net-(A2-Pad17)
- A2 pad 18: (no net) -> Net-(A2-Pad18)
- A2 pad 19: (no net) -> /a0
- A2 pad 2: (no net) -> Net-(A2-Pad2)
- A2 pad 20: (no net) -> /a1
- A2 pad 21: (no net) -> /a2
- A2 pad 22: (no net) -> /a3
- A2 pad 23: (no net) -> /a4
- A2 pad 24: (no net) -> /a5
- A2 pad 25: (no net) -> /a6
- A2 pad 26: (no net) -> /a7
- A2 pad 27: (no net) -> /5v
- A2 pad 28: (no net) -> Net-(A2-Pad28)
- A2 pad 29: (no net) -> /gnd
- A2 pad 3: (no net) -> Net-(A2-Pad3)
- A2 pad 30: (no net) -> /vin
- A2 pad 4: (no net) -> /gnd
- A2 pad 5: (no net) -> /d2
- A2 pad 6: (no net) -> /d3
- A2 pad 7: (no net) -> /d4
- A2 pad 8: (no net) -> /d5
- A2 pad 9: (no net) -> /d6
- A3 pad 3: (no net) -> /a5
- A3 pad 4: (no net) -> /a4
- A3 pad 5: (no net) -> /5v
- A3 pad 6: (no net) -> /gnd
- J1 pad 1: (no net) -> Net-(J1-Pad1)
- J1 pad 10: (no net) -> /d5
- J1 pad 11: (no net) -> /d6
- J1 pad 12: (no net) -> /d10
- J1 pad 13: (no net) -> /5v
- J1 pad 14: (no net) -> /gnd
- J1 pad 15: (no net) -> /a0
- J1 pad 16: (no net) -> /a1
- J1 pad 17: (no net) -> /a2
- J1 pad 18: (no net) -> /a3
- J1 pad 19: (no net) -> /a6
- J1 pad 2: (no net) -> /In-
- J1 pad 20: (no net) -> /a7
- J1 pad 3: (no net) -> /5v
- J1 pad 4: (no net) -> /gnd
- J1 pad 5: (no net) -> /a5
- J1 pad 6: (no net) -> /a4
- J1 pad 7: (no net) -> /d2
- J1 pad 8: (no net) -> /d3
- J1 pad 9: (no net) -> /d4
- J2 pad 1: (no net) -> Net-(J2-Pad1)
- J2 pad 2: (no net) -> Net-(J2-Pad2)
- J2 pad 3: (no net) -> Net-(J2-Pad3)
- J2 pad 4: (no net) -> Net-(J2-Pad4)
- J2 pad 5: (no net) -> Net-(J2-Pad5)
- J2 pad 6: (no net) -> Net-(J2-Pad6)
- J2 pad 7: (no net) -> Net-(J2-Pad7)
- J2 pad 8: (no net) -> /d7
- J4 pad 1: (no net) -> Net-(J4-Pad1)
- J4 pad 2: (no net) -> Net-(J4-Pad2)
- J4 pad 3: (no net) -> Net-(J4-Pad3)
- J4 pad 4: (no net) -> Net-(J4-Pad4)
- J4 pad 5: (no net) -> Net-(J4-Pad5)
- J4 pad 6: (no net) -> Net-(J4-Pad6)
- J5 pad 1: (no net) -> Net-(J5-Pad1)
- J5 pad 2: (no net) -> Net-(J5-Pad2)
- J5 pad 3: (no net) -> /gnd
- J5 pad 4: (no net) -> /5v
- J5 pad 5: (no net) -> Net-(J5-Pad5)
- J5 pad 6: (no net) -> Net-(J5-Pad6)
- J5 pad 7: (no net) -> Net-(J5-Pad7)
- J5 pad 8: (no net) -> Net-(J5-Pad8)
Routing:
- net /5v: track 0.00 -> 224.1 mm
- net /gnd: track 0.00 -> 220.6 mm
- net /a4: track 0.00 -> 117.6 mm
- net /a5: track 0.00 -> 117.0 mm
- net /a6: track 0.00 -> 85.3 mm
- net /a3: track 0.00 -> 77.8 mm
- net /a7: track 0.00 -> 77.5 mm
- net /a2: track 0.00 -> 76.3 mm
- net /a1: track 0.00 -> 76.0 mm
- net /a0: track 0.00 -> 75.1 mm
- net /vin: track 0.00 -> 69.3 mm
- net /d2: track 0.00 -> 67.6 mm
- net /d3: track 0.00 -> 64.0 mm
- net /d4: track 0.00 -> 59.4 mm
- net /d5: track 0.00 -> 55.5 mm
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Other:
- net class Default: clearance 0.2 -> 0.25; trace_width 0.25 -> 0.45
- rule pad_to_mask_clearance: 0.051 -> 0.05
- rule solder_mask_min_width: 0.25 -> 0.2
- rule trace_clearance: 0.2 -> 0.25
- board text added: "+"
- board text added: "-"
- board text added: "5V"
- board text added: "A0"
- board text added: "A1"
- board text added: "A2"
- board text added: "A3"
- board text added: "A5"
- board text added: "A6"
- board text added: "A7"
- board text added: "D10"
- board text added: "D2"
- board text added: "D3"
- board text added: "D4"
- board text added: "D5"
- board text added: "D6"
- board text added: "D7"
- board text added: "D8"
- board text added: "D9"
- board text added: "GND"

Commit message: Проект окочен
Routing:
- net /5v: track 224.1 -> 172.4 mm
- net /gnd: track 220.6 -> 190.6 mm
- net /a7: track 77.5 -> 83.3 mm
- net /a2: track 76.3 -> 72.2 mm
- net /a0: track 75.1 -> 78.2 mm
- net /a1: track 76.0 -> 79.1 mm
- net /a3: track 77.8 -> 74.9 mm
- net /a6: track 85.3 -> 82.5 mm
