File: Second/project/galvo-schematic.sch (KiCad schematic (older format))
At the start: 19 parts, among them IC1 TL082P, IC2 TL082P, J1 0022272031, X2 JST-XH-03-PIN-ROUND-PAD, X3 JST-XH-03-PIN-ROUND-PAD

Commit message: Переработка проекта 2
Parts:
- removed IC1, IC2: TL082P, galvo-schematic:DIL08, symbol galvo-schematic-eagle-import:TL082P
- added U1: TL084IPT, Package_SO:TSSOP-14_4.4x5mm_P0.65mm, symbol Amplifier_Operational:TL084
- renumbered DAC to U2
Connections:
- net +V15: now also U1.4 (V+)
- net -V15: now also U1.11 (V-)
- net GND: now also U1.12 (+), U1.5 (+)
- net ILDAX+15V: now also U1.1
- net ILDAX-15V: now also U1.7
- net ILDAY+15V: now also U1.8
- net ILDAY-15V: now also U1.14
- net at R12.1, R3.2: now also U1.13 (-)
- net at R1.2, Y-GAIN1.E: now also U1.9 (-)
- net at Y-OFFSET1.S: now also U1.10 (+)
- net at R5.2, X-GAIN1.E: now also U1.2 (-)
- net at R11.1, R7.2: now also U1.6 (-)
- net at X-OFFSET1.S: now also U1.3 (+)
Changed lines of the file:
@@
 $EndDescr
-Wire Wire Line
-	3200 7500 3550 7500
 Wire Wire Line
 	10900 3600 10800 3600
@@
 ILDAX+15V
 Wire Wire Line
-	7500 7100 7500 6800
-Wire Wire Line
-	7500 6800 6900 6800
-Wire Wire Line
-	8300 6000 8300 7100
-Wire Wire Line
-	8300 7100 7500 7100
-Connection ~ 7500 7100
-Text Label 7200 6800 0    70   ~ 0
+	6900 6350 6900 6800
+Text Label 6900 6350 1    70   ~ 0
 +V15
 Wire Wire Line
@@
 Wire Wire Line
 	7000 3300 7000 1600
-Wire Wire Line
-	5900 3500 5900 3300
-Connection ~ 5900 3300
 Text Label 5550 2800 0    70   ~ 0
 +V15
@@
 Text Label 7500 1600 3    70   ~ 0
 +V15
-Wire Wire Line
-	7500 7700 8100 7700
-Wire Wire Line
-	8100 7700 8100 6000
-Text Label 8100 6000 1    70   ~ 0
--V15
-Wire Wire Line
-	6800 4100 6800 1600
-Wire Wire Line
-	5900 4100 6800 4100
-Text Label 6800 1600 1    70   ~ 0
--V15
 Wire Wire Line
 	7900 1500 7900 1600
@@
 GND
 Wire Wire Line
-	8200 6000 8200 7200
-Wire Wire Line
 	8200 7200 8200 8300
 Wire Wire Line
@@
 	9100 7200 8200 7200
 Connection ~ 8200 8300
-Text Label 8200 6000 1    70   ~ 0
-GND
-Connection ~ 8200 7200
 Text Label 8200 8500 3    70   ~ 0
 GND
@@
 $EndComp
 $Comp
-L galvo-schematic-eagle-import:TL082P IC1
-U 1 0 22F7723E
-P 7500 7400
-F 0 "IC1" H 7600 7525 59  0001 L BNN
-F 1 "TL082P" H 7600 7200 59  0001 L BNN
-F 2 "galvo-schematic:DIL08" H 7500 7400 50  0001 C CNN
-F 3 "" H 7500 7400 50  0001 C CNN
-	1    7500 7400
-	1    0    0    -1
-$EndComp
-$Comp
-L galvo-schematic-eagle-import:TL082P IC1
-U 2 0 22F77232
-P 9400 7300
-F 0 "IC1" H 9500 7425 59  0001 L BNN
-F 1 "TL082P" H 9500 7100 59  0001 L BNN
-F 2 "galvo-schematic:DIL08" H 9400 7300 50  0001 C CNN
-F 3 "" H 9400 7300 50  0001 C CNN
-	2    9400 7300
-	1    0    0    -1
-$EndComp
-$Comp
-L galvo-schematic-eagle-import:TL082P IC1
-U 3 0 22F77236
-P 7500 7400
-F 0 "IC1" H 7600 7525 59  0001 L BNN
-F 1 "TL082P" H 7600 7200 59  0001 L BNN
-F 2 "galvo-schematic:DIL08" H 7500 7400 50  0001 C CNN
-F 3 "" H 7500 7400 50  0001 C CNN
-	3    7500 7400
-	1    0    0    -1
-$EndComp
-$Comp
 L galvo-schematic-eagle-import:R-EU_0207_10 R5
 U 1 0 4373A00B
@@
 $EndComp
 $Comp
-L galvo-schematic-eagle-import:TL082P IC2
-U 1 0 BC34DC86
-P 5900 3800
-F 0 "IC2" H 6000 3925 59  0001 L BNN
-F 1 "TL082P" H 6000 3600 59  0001 L BNN
-F 2 "galvo-schematic:DIL08" H 5900 3800 50  0001 C CNN
-F 3 "" H 5900 3800 50  0001 C CNN
-	1    5900 3800
-	1    0    0    -1
-$EndComp
-$Comp
-L galvo-schematic-eagle-import:TL082P IC2
-U 2 0 BC34DC8A
-P 8200 3700
-F 0 "IC2" H 8300 3825 59  0001 L BNN
-F 1 "TL082P" H 8300 3500 59  0001 L BNN
-F 2 "galvo-schematic:DIL08" H 8200 3700 50  0001 C CNN
-F 3 "" H 8200 3700 50  0001 C CNN
-	2    8200 3700
-	1    0    0    -1
-$EndComp
-$Comp
-L galvo-schematic-eagle-import:TL082P IC2
-U 3 0 BC34DC8E
-P 5900 3800
-F 0 "IC2" H 6000 3925 59  0001 L BNN
-F 1 "TL082P" H 6000 3600 59  0001 L BNN
-F 2 "galvo-schematic:DIL08" H 5900 3800 50  0001 C CNN
-F 3 "" H 5900 3800 50  0001 C CNN
-	3    5900 3800
-	1    0    0    -1
-$EndComp
-$Comp
 L galvo-schematic-eagle-import:MA06-1 SV4
 U 1 0 52E1D252
@@
 Wire Wire Line
 	6800 8500 7200 8500
-Text Label 7000 1600 1    70   ~ 0
-+V15
-Text Label 8300 6000 1    70   ~ 0
-+V15
 NoConn ~ 7500 6300
 NoConn ~ 5900 2200
 $Comp
-L Analog_DAC:MCP4822 DAC
+L Analog_DAC:MCP4822 U2
 U 1 1 5C94B8C6
 P 2550 3900
-F 0 "DAC" H 2150 4400 50  0000 C CNN
+F 0 "U2" H 2150 4400 50  0000 C CNN
 F 1 "MCP4822" H 2250 4300 50  0000 C CNN
 F 2 "Package_SO:MSOP-8_3x3mm_P0.65mm" H 3350 3600 50  0001 C CNN
@@
 Wire Wire Line
 	3550 4100 3550 7500
-Connection ~ 3550 7500
 Wire Wire Line
 	3550 7500 6200 7500
+$Comp
+L Amplifier_Operational:TL084 U1
+U 1 1 5C955528
+P 5900 3800
+F 0 "U1" H 5725 4150 50  0000 C CNN
+F 1 "TL084IPT" H 5725 4075 50  0000 C CNN
+F 2 "Package_SO:TSSOP-14_4.4x5mm_P0.65mm" H 5850 3900 50  0001 C CNN
+F 3 "http://www.ti.com/lit/ds/symlink/tl081.pdf" H 5950 4000 50  0001 C CNN
+	1    5900 3800
+	1    0    0    -1
+$EndComp
+$Comp
+L Amplifier_Operational:TL084 U1
+U 2 1 5C9556F9
+P 8200 3700
+F 0 "U1" H 8200 4067 50  0000 C CNN
+F 1 "TL084IPT" H 8200 3976 50  0000 C CNN
+F 2 "" H 8150 3800 50  0001 C CNN
+F 3 "http://www.ti.com/lit/ds/symlink/tl081.pdf" H 8250 3900 50  0001 C CNN
+	2    8200 3700
+	1    0    0    -1
+$EndComp
+$Comp
+L Amplifier_Operational:TL084 U1
+U 3 1 5C955911
+P 7500 7400
+F 0 "U1" H 7500 7767 50  0000 C CNN
+F 1 "TL084IPT" H 7500 7676 50  0000 C CNN
+F 2 "" H 7450 7500 50  0001 C CNN
+F 3 "http://www.ti.com/lit/ds/symlink/tl081.pdf" H 7550 7600 50  0001 C CNN
+	3    7500 7400
+	1    0    0    -1
+$EndComp
+$Comp
+L Amplifier_Operational:TL084 U1
+U 4 1 5C95598A
+P 9400 7300
+F 0 "U1" H 9400 7667 50  0000 C CNN
+F 1 "TL084IPT" H 9400 7576 50  0000 C CNN
+F 2 "" H 9350 7400 50  0001 C CNN
+F 3 "http://www.ti.com/lit/ds/symlink/tl081.pdf" H 9450 7500 50  0001 C CNN
+	4    9400 7300
+	1    0    0    -1
+$EndComp
+$Comp
+L Amplifier_Operational:TL084 U1
+U 5 1 5C959962
+P 6000 3800
+F 0 "U1" H 6000 3650 50  0001 L CNN
+F 1 "TL084IPT" H 6000 3550 50  0001 L CNN
+F 2 "" H 5950 3900 50  0001 C CNN
+F 3 "http://www.ti.com/lit/ds/symlink/tl081.pdf" H 6050 4000 50  0001 C CNN
+	5    6000 3800
+	1    0    0    -1
+$EndComp
+Wire Wire Line
+	6800 4100 6800 1600
+Wire Wire Line
+	5900 4100 6800 4100
+Connection ~ 5900 3300
+Wire Wire Line
+	5900 3500 5900 3300
+Text Label 6800 1600 1    70   ~ 0
+-V15
+Text Label 7000 1600 1    70   ~ 0
++V15
 $EndSCHEMATC
