File: Second/project/galvo-schematic.kicad_pcb (KiCad board)
At the start: 2 copper layers, 30.5 x 32 mm, 23 parts, among them IC1 TL082P, IC2 TL082P, J1 0022272031, X2 JST-XH-03-PIN-ROUND-PAD, X3 JST-XH-03-PIN-ROUND-PAD

Commit message: Переработка проекта 2
Parts:
- removed DAC: MCP4822, Package_SO:MSOP-8_3x3mm_P0.65mm
- removed IC1, IC2: TL082P, galvo-schematic:DIL08
- removed X-OFFS.1, Y-OFFS.1: 10k, galvo-schematic:Potentiometer_Murata_PVS3_Vertical
- added U1: TL084, Package_SO:TSSOP-14_4.4x5mm_P0.65mm, F.Cu at (128.3, 92.5)
- added U2: MCP4822, Package_SO:MSOP-8_3x3mm_P0.65mm, F.Cu at (128.0, 101.9)
- added X-OFFSET1: 10k, galvo-schematic:Potentiometer_Murata_PVS3_Vertical, F.Cu at (136.1, 97.5)
- added Y-OFFSET1: 10k, galvo-schematic:Potentiometer_Murata_PVS3_Vertical, F.Cu at (136.1, 85.3)
- J1: footprint galvo-schematic:KK6410-2031_3-PIN -> Connector_Molex:Molex_KK-254_AE-6410-03A_1x03_P2.54mm_Vertical
- X2, X3: footprint galvo-schematic:JST-XH-03-PACKAGE-ROUND-PAD -> Connector_JST:JST_XH_B03B-XH-A_1x03_P2.50mm_Vertical
- moved R11 9.92 mm to (124.2, 106.7)
- moved R12 9.18 mm to (124.2, 95.8)
- moved R1 7.73 mm to (132.8, 90.2)
- moved X-GAIN1 7.22 mm to (136.1, 103.6)
- moved R6 4.96 mm to (137.2, 98.8)
- moved J1 4.83 mm to (132.8, 110.2)
- moved R5 4.49 mm to (132.6, 102.4), turned to 0 degrees
- moved R2 3.42 mm to (137.3, 86.6)
- moved Y-GAIN1 3.33 mm to (136.1, 91.4)
- moved R7 2.84 mm to (124.2, 102.1)
- moved X2 2.67 mm to (119.9, 105.7), turned to 90 degrees
- moved X3 2.67 mm to (119.9, 95.0), turned to 90 degrees
- moved R3 2.41 mm to (124.2, 91.4), turned to 0 degrees
Routing:
- net /+V15: track 66.5 -> 37.4 mm, vias 1 -> 0
- net /-V15: track 24.8 -> 0.00 mm
- net Net-(DAC1-Pad6): track 14.5 -> 0.00 mm, vias 1 -> 0
- net +5V: track 6.66 -> 20.7 mm
- net /LATCH: track 22.5 -> 35.9 mm, vias 1 -> 0
- net /SCK: track 11.4 -> 24.7 mm
- net /CS: track 9.51 -> 22.8 mm
- net Net-(U1-Pad10): track 0.00 -> 12.9 mm
- net /SDI: track 13.8 -> 26.5 mm
- net Net-(R5-Pad2): track 9.79 -> 22.1 mm, vias 0 -> 2
- net Net-(IC1-Pad3): track 11.4 -> 0.00 mm, vias 1 -> 0
- net Net-(U1-Pad3): track 0.00 -> 11.4 mm
- net Net-(R11-Pad1): track 8.92 -> 19.7 mm, vias 0 -> 1
- net Net-(R6-Pad2): track 12.9 -> 2.83 mm
- net Net-(R1-Pad2): track 23.0 -> 13.4 mm, vias 1 -> 2
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Other:
- board text added: "MCP4822"

Commit message: Предварительно закончен второй проект
Parts:
- removed the REF** at (119.9, 84.8)
- removed the REF** at (119.9, 110.7)
- removed the REF** at (144.3, 84.8)
- removed X-GAIN1: 10k, galvo-schematic:Potentiometer_Murata_PVS3_Vertical
- added REF**: MountingHole_2.5mm, MountingHole:MountingHole_2.5mm, F.Cu at (124.5, 84.8)
- added REF**: MountingHole_2.5mm, MountingHole:MountingHole_2.5mm, F.Cu at (146.1, 84.8)
- added X-GAIN: 10k, galvo-schematic:Potentiometer_Murata_PVS3_Vertical, F.Cu at (130.0, 102.9)
- moved J1 25.0 mm to (135.1, 85.3), turned to 0 degrees
- moved X2 21.4 mm to (140.7, 110.7), turned to 180 degrees
- moved X3 18.7 mm to (130.0, 110.7), turned to 180 degrees
- moved R11 17.8 mm to (142.0, 107.4), turned to 270 degrees
- moved R3 16.2 mm to (126.5, 107.4), turned to 90 degrees
- moved R7 14.0 mm to (137.2, 107.4), turned to 90 degrees
- moved R12 13.7 mm to (131.3, 107.5), turned to 270 degrees
- moved U1 10.7 mm to (138.7, 94.7)
- moved U2 10.4 mm to (138.4, 102.4)
- moved R1 6.14 mm to (126.7, 89.4)
- moved R6 6.14 mm to (131.1, 98.0)
- moved X-OFFSET 6.14 mm to (130.0, 96.8)
- moved Y-GAIN 6.14 mm to (130.0, 90.7)
- moved Y-OFFSET 6.14 mm to (130.0, 84.6)
- moved R2 6.14 mm to (131.2, 85.9)
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- renumbered X-OFFSET1 to X-OFFSET, Y-GAIN1 to Y-GAIN, Y-OFFSET1 to Y-OFFSET
Routing:
- net /ILDAY-15V: track 3.60 -> 37.9 mm, vias 0 -> 1
- net Net-(DAC1-Pad6): track 0.00 -> 22.7 mm, vias 0 -> 1
- net /ILDAX-15V: track 3.71 -> 23.2 mm
- net /SDI: track 26.5 -> 7.72 mm
- net /SCK: track 24.7 -> 6.44 mm
- net /LATCH: track 35.9 -> 17.8 mm
- net /CS: track 22.8 -> 5.66 mm
- net Net-(R12-Pad1): track 12.4 -> 28.7 mm
- net /ILDAX+15V: track 21.9 -> 37.1 mm
- net +5V: track 20.7 -> 6.24 mm
- net /ILDAY+15V: track 27.8 -> 41.6 mm
- net /+V15: track 37.4 -> 26.7 mm, vias 0 -> 1
- net Net-(U1-Pad10): track 12.9 -> 18.8 mm
- net Net-(DAC1-Pad8): track 8.62 -> 13.6 mm
- net GND: track 4.61 -> 8.84 mm, vias 3 -> 4
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Other:
- board size 30.5 x 32 mm -> 27.7 x 32 mm
- board text added: "+"
- board text added: "+5v"
- board text added: "-"
- board text added: "CS"
- board text added: "LDAC"
- board text added: "SCK"
- board text added: "SDI"

Commit message: Очередная корректировка проекта
Удалена шелкография номиналов резисторов.
Заменен потенциометр.
Parts:
- renumbered X-OFFSET to X-OFFS, Y-OFFSET to Y-OFFS
Routing:
- net GND: track 8.84 -> 9.47 mm

Commit message: Закончен 2 проект
Parts:
- R1, R5: footprint Resistor_SMD:R_2010_5025Metric_Pad1.52x2.65mm_HandSolder -> Resistor_SMD:R_0805_2012Metric_Pad1.15x1.40mm_HandSolder
Routing:
- net Net-(R1-Pad2): track 15.6 -> 17.1 mm
- net Net-(R5-Pad2): track 21.0 -> 22.3 mm
- net Net-(DAC1-Pad8): track 13.6 -> 12.3 mm
- net Net-(DAC1-Pad6): track 22.7 -> 23.7 mm
